File: hardware/PCB/pill_box/pill_box.kicad_sch (KiCad schematic)
At the start: 22 parts, among them J1 MOTOR DRIVER 1, J10 Conn_01x15_Pin, J11 3.3v, J12 5v, J13 Conn_01x15_Pin, J2 MOTOR DRIVER 2, J3 MOTOR DRIVER 3, J4 SERVO MOTOR, J5 LED 1, J6 LED 2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

Commit message: capacitor
Parts:
- added C1, C2: 100uF, Capacitor_THT:CP_Radial_D8.0mm_P3.50mm, symbol Device:C_Polarized
- added C3, C4, C5: 0.1uF, Capacitor_THT:C_Disc_D5.0mm_W2.5mm_P2.50mm, symbol Device:C
- J10: value Conn_01x15_Pin -> node mcu
- J13: value Conn_01x15_Pin -> node mcu_second
Connections:
- net D2(GPIO4) is gone; now on net +3.3V: J13.3 (Pin_3), R1.2, R3.2, U2.14 (SCL), U3.14 (SCL)
- net +3.3V: now also C1.1, C3.1, C4.1
- net +5V: now also C2.1
- net 3.3V: now also C5.1
- net GND: now also C1.2, C2.2, C3.2, C4.2, C5.2
- no-connect marks 23 -> 22
